File: 03_Hardware/Drucksensor.kicad_sch (KiCad schematic)
At the start: 99 parts, among them J103 Conn_01x02, J110 DS18B20, J111 Conn_01x06_Male, Q1 BC817, SW103 SW_DIP_x08, U103 ATmega8A-A, U104 REF3040, U105 74HC165, U107 SN75176AD, U108 CAT24M01W, Y101 16MHz

Commit message: Versionsänderungen 6.99 auf 7.0rc, Übergang alte Version 1 auf Version 2.dev
Parts:
- removed ?: (no value), symbol Connector:Conn_01x03_Male
- removed ? (x5): (no value), symbol Device:R
- removed ?: (no value), symbol Device:Fuse
- removed ? (x4): (no value), symbol Device:C
- removed ? (x2): (no value), symbol Connector:Conn_01x02_Male
- removed ?: (no value), symbol Reference_Voltage:REF3040
- removed ?: (no value), symbol MCU_Module:Arduino_UNO_R3
- removed ?: (no value), symbol Connector:DB15_Female_MountingHoles
- added J114: AVR-ISP-6, Connector_IDC:IDC-Header_2x03_P2.54mm_Vertical, symbol Connector:AVR-ISP-6
- added R102: 1k, Resistor_SMD:R_0603_1608Metric, symbol Device:R
- C101: renamed from C125; value 100p -> paar nF; footprint (none) -> Capacitor_SMD:C_0603_1608Metric
- C108, C109: renamed from ?; value (none) -> 1u; footprint (none) -> Capacitor_SMD:C_0603_1608Metric
- C110, C111: renamed from ?; value (none) -> 470n; footprint (none) -> Capacitor_SMD:C_0603_1608Metric
- C114, C125: footprint (none) -> Capacitor_SMD:C_0603_1608Metric
- C115, C119, C120, C122, C124: renamed from C114; footprint (none) -> Capacitor_SMD:C_0603_1608Metric
- C116, C117, C118: renamed from C114; value 100n -> 1u; footprint (none) -> Capacitor_SMD:C_0603_1608Metric
- C121, C123: renamed from C114; value 100n -> 22u; footprint (none) -> Capacitor_SMD:C_1206_3216Metric
- C126, C127, C128: renamed from C125; footprint (none) -> Capacitor_SMD:C_0603_1608Metric
- C129, C130: renamed from ?; value (none) -> 100n; footprint (none) -> Capacitor_SMD:C_0603_1608Metric
- D103: renamed from ?; value (none) -> STPS340U; footprint (none) -> Diode_SMD:D_SMB
- D105: value D_Schottky -> STPS340U; footprint (none) -> Diode_SMD:D_SMB
- F102, F103, F104: renamed from ?; value (none) -> Fuse; footprint (none) -> Resistor_SMD:R_1210_3225Metric
- J101: renamed from ?; value (none) -> 24V in; footprint (none) -> Connector_JST:JST_XH_B2B-XH-A_1x02_P2.50mm_Vertical
- J103: value Conn_01x02 -> RS485-mini-1; footprint (none) -> Connector_JST:JST_XH_B2B-XH-AM_1x02_P2.50mm_Vertical
- J104, J108, J109, J112: renamed from ?; value (none) -> RJ45; footprint (none) -> Sven:RJ45_Amphenol_54602_mod
- J110: footprint (none) -> Connector_JST:JST_XH_B3B-XH-AM_1x03_P2.50mm_Vertical
- J111: value Conn_01x06_Male -> BMP280; footprint (none) -> Connector_PinHeader_2.54mm:PinHeader_1x06_P2.54mm_Vertical
- J113: renamed from J103; value Conn_01x02 -> RS485-mini-1; footprint (none) -> Connector_JST:JST_XH_B2B-XH-AM_1x02_P2.50mm_Vertical
- JP101: value Jumper_2_Open -> 24V_ext; footprint (none) -> Connector_PinHeader_2.54mm:PinHeader_1x02_P2.54mm_Vertical
- JP102: renamed from JP101; value Jumper_2_Open -> 5V_ext; footprint (none) -> Connector_PinHeader_2.54mm:PinHeader_1x02_P2.54mm_Vertical
- JP103: footprint (none) -> Connector_PinHeader_2.54mm:PinHeader_1x02_P2.54mm_Vertical
- NT101: footprint (none) -> NetTie:NetTie-2_SMD_Pad0.5mm
- R101, R126: renamed from R125; value R -> 15R; footprint (none) -> Resistor_SMD:R_1206_3216Metric
- R103, R104: renamed from ?; value (none) -> 24k 1%; footprint (none) -> Resistor_SMD:R_0603_1608Metric
- R109, R115: renamed from ?; value (none) -> 20k 1%; footprint (none) -> Resistor_SMD:R_0603_1608Metric
- R110, R114: renamed from ?; value (none) -> 33k 1%; footprint (none) -> Resistor_SMD:R_0603_1608Metric
- R111, R137: renamed from ?; value (none) -> 33k; footprint (none) -> Resistor_SMD:R_0603_1608Metric
- R112, R138: renamed from ?; value (none) -> NC; footprint (none) -> Resistor_SMD:R_1206_3216Metric; now not fitted
- R113, R139: renamed from ?; value (none) -> 1k; footprint (none) -> Resistor_SMD:R_0603_1608Metric
- R125: value R -> 10k; footprint (none) -> Resistor_SMD:R_0603_1608Metric
- R127: footprint (none) -> Resistor_SMD:R_0603_1608Metric
- R128: renamed from R127; footprint (none) -> Resistor_SMD:R_0603_1608Metric
- R129: renamed from R127; value 100k -> 4,7k; footprint (none) -> Resistor_SMD:R_0603_1608Metric
- R130: renamed from R127; value 100k -> 10k; footprint (none) -> Resistor_SMD:R_0603_1608Metric
- R131, R132, R133, R134: renamed from R127; value 100k -> tbd; footprint (none) -> Resistor_SMD:R_0603_1608Metric
- R135, R136: renamed from R127; value 100k -> 3,3k; footprint (none) -> Resistor_SMD:R_0603_1608Metric
- RN101, RN102: renamed from RN201; value R_Pack04 -> 56k; footprint (none) -> Resistor_SMD:R_Array_Convex_4x1206
- TP101: value TestPoint -> Pin_7; footprint (none) -> TestPoint:TestPoint_Keystone_5005-5009_Compact
- TP102: renamed from TP101; value TestPoint -> Pin_8; footprint (none) -> TestPoint:TestPoint_Keystone_5005-5009_Compact
- U105: footprint (none) -> Package_SO:SOIC-16_3.9x9.9mm_P1.27mm
- U106: renamed from ?; value (none) -> 74HC595; footprint (none) -> Package_SO:SOIC-16_3.9x9.9mm_P1.27mm
- Y101: footprint (none) -> Crystal:Resonator_SMD_Murata_CSTxExxV-3Pin_3.0x1.1mm
- renumbered D102 to D106, Q1 to Q2
Connections:
- net +3V3: now also R130.2, U108.8 (VCC)
- net +5V: now also J114.2 (VCC); no longer R130.2, U108.8 (VCC)
- net GND: now also J114.6 (GND)
- net MISO_Schieber_Daten_In: now also J114.1 (MISO), R102.2; no longer U105.9 (Q7)
- net MOSI_Schieber_Daten_Out: now also J114.4 (MOSI)
- net Reset: now also J114.5 (~{RST})
- net SCK_Schieber_Takt: now also J114.3 (SCK)
- new net: R102.1, U105.9 (Q7)
- no-connect marks 19 -> 9
Other:
- note added: "Ausgang hat keinen High-Z-Modus -> muss im Fall des programmierens vom Progger überdrückt werden können!"
- note added: "ESD-Schutz an ID-Widerstandsmessungen fehlen!"
- note added: "bei Speichermangel: mega328pb verwenden!"
