File: 03_Hardware/Drucksensor.kicad_pcb (KiCad board)
At the start: 2 copper layers, 99 x 67 mm, 99 parts, among them J101 Conn_01x02, J102 Start, J103 RJ45, J104 RJ45, J105 DB15_Female_MountingHoles, J106 Serial, J107 Conn_01x03_Male, Q101 Q_NMOS_GSD, Q102 Q_NMOS_GSD, Q103 Q_NMOS_GSD, SW101 SW_DPST, SW102 SW_SPDT, U101 REF3040, U102 MAX232, U201 KCSA02-106, U202 74HC595, U203 KCSA02-106, U204 74HC595, U205 KCSA02-106, U206 74HC595, U207 KCSA02-106, U208 74HC595

Commit message: Reste von altem Projekt gelöscht und neue Daten, so fertig, eingefügt.
Parts:
- removed A101: Arduino_UNO_R3, Module:Arduino_UNO_R3
- removed C102, C103, C104, C105: 1µ 16V, Capacitor_SMD:C_0805_2012Metric
- removed C106, C107, C112, C113: 100n, Capacitor_SMD:C_0603_1608Metric
- removed F101: Fuse, Resistor_SMD:R_1210_3225Metric
- removed J102: Start, Connector_PinSocket_2.54mm:PinSocket_1x02_P2.54mm_Vertical
- removed J104: RJ45, Sven:RJ45_Amphenol_54602_mod
- removed J105: DB15_Female_MountingHoles, Connector_Dsub:DSUB-15_Female_Vertical_P2.77x2.84mm_MountingHoles
- removed J106: Serial, Connector_PinSocket_2.54mm:PinSocket_1x02_P2.54mm_Vertical
- removed J107: Conn_01x03_Male, Connector_PinSocket_2.54mm:PinSocket_1x03_P2.54mm_Vertical
- removed Q101, Q102, Q103: Q_NMOS_GSD, Package_TO_SOT_SMD:SOT-23
- removed R105, R116, R123, R124: Open, Resistor_SMD:R_0805_2012Metric
- removed R106, R107, R108, R118, R119, R120, R122: 10k, Resistor_SMD:R_0603_1608Metric
- removed R117, R121: 10, Resistor_SMD:R_0603_1608Metric
- removed R207, R208, R209, R210, R211, R212, R213, R214, R215, R216, R217, R218, R219, R220, R221, R222, R223, R224, R225, R226, R227, R228, R229, R230, R231, R232: R, Resistor_SMD:R_0805_2012Metric
- removed SW101: SW_DPST, Sven:Switch_DPDT
- removed SW102: SW_SPDT, Sven:Switch_DPDT
- removed U101: REF3040, Package_TO_SOT_SMD:SOT-23
- removed U102: MAX232, Package_SO:SOIC-16W_7.5x10.3mm_P1.27mm
- added C114: 100n, Capacitor_SMD:C_0603_1608Metric, F.Cu at (204.4, 29.1)
- added C115: 100n, Capacitor_SMD:C_0603_1608Metric, F.Cu at (204.4, 31.6)
- added C116: 1u, Capacitor_SMD:C_0603_1608Metric, F.Cu at (204.4, 34.1)
- added C117: 1u, Capacitor_SMD:C_0603_1608Metric, F.Cu at (204.4, 36.6)
- added C118: 1u, Capacitor_SMD:C_0603_1608Metric, F.Cu at (204.4, 39.1)
- added C119: 100n, Capacitor_SMD:C_0603_1608Metric, F.Cu at (204.4, 41.6)
- added C120: 100n, Capacitor_SMD:C_0603_1608Metric, F.Cu at (204.4, 44.1)
- added C121: 22u, Capacitor_SMD:C_1206_3216Metric, F.Cu at (215.4, 57.4)
- added C122: 100n, Capacitor_SMD:C_0603_1608Metric, F.Cu at (204.4, 46.6)
- added C123: 22u, Capacitor_SMD:C_1206_3216Metric, F.Cu at (215.4, 60.7)
- added C124: 100n, Capacitor_SMD:C_0603_1608Metric, F.Cu at (208.4, 29.1)
- added C125: 100p, Capacitor_SMD:C_0603_1608Metric, F.Cu at (208.4, 31.6)
- added C126: 100p, Capacitor_SMD:C_0603_1608Metric, F.Cu at (208.4, 34.1)
- added C127: 100p, Capacitor_SMD:C_0603_1608Metric, F.Cu at (208.4, 36.6)
- added C128: 100p, Capacitor_SMD:C_0603_1608Metric, F.Cu at (208.4, 39.1)
- added C129: 100n, Capacitor_SMD:C_0603_1608Metric, F.Cu at (208.4, 41.6)
- added C130: 100n, Capacitor_SMD:C_0603_1608Metric, F.Cu at (208.4, 44.1)
- added C201: 100n, Resistor_SMD:R_0603_1608Metric, F.Cu at (237.6, 82.6)
- added C202: 100n, Resistor_SMD:R_0603_1608Metric, F.Cu at (237.6, 85.1)
- added C203: 100n, Resistor_SMD:R_0603_1608Metric, F.Cu at (237.6, 87.6)
- added C204: 100n, Resistor_SMD:R_0603_1608Metric, F.Cu at (237.6, 90.2)
- added C205: 100n, Resistor_SMD:R_0603_1608Metric, F.Cu at (237.6, 92.7)
- added C206: 100n, Resistor_SMD:R_0603_1608Metric, F.Cu at (237.6, 95.2)
- added C301: 10u 16V, Capacitor_SMD:C_1206_3216Metric, F.Cu at (257.3, 29.5)
- added C302: 10u 16V, Capacitor_SMD:C_1206_3216Metric, F.Cu at (257.3, 32.8)
- added C303: 100n, Capacitor_SMD:C_0603_1608Metric, F.Cu at (252.4, 29.1)
- added C304: 10u 25V, Capacitor_SMD:C_1206_3216Metric, F.Cu at (257.3, 36.2)
- added C305: 22u, Capacitor_SMD:C_1206_3216Metric, F.Cu at (257.3, 39.5)
- added C306: 22u, Capacitor_SMD:C_1206_3216Metric, F.Cu at (257.3, 42.9)
- added C307: 75p, Capacitor_SMD:C_0603_1608Metric, F.Cu at (252.4, 31.6)
- added C308: 100u 50V, Capacitor_THT:CP_Radial_D8.0mm_P3.50mm, F.Cu at (263.3, 40.8)
- added D102: SM6T30A, Diode_SMD:D_SMB, F.Cu at (211.2, 66.9)
- added D104: SD05_SOD323, Diode_SMD:D_SOD-323, F.Cu at (245.4, 50.5)
- added D201: rot, LED_THT:LED_Rectangular_W3.0mm_H2.0mm, F.Cu at (204.0, 83.2)
- added D202: rot, LED_THT:LED_Rectangular_W3.0mm_H2.0mm, F.Cu at (204.0, 87.0)
- added D203: grün, LED_THT:LED_D5.0mm, F.Cu at (204.8, 77.6)
- added D204: grün, LED_THT:LED_D5.0mm, F.Cu at (212.3, 77.6)
- added D205: grün, LED_THT:LED_D5.0mm, F.Cu at (219.8, 77.6)
- added D206: grün, LED_THT:LED_D5.0mm, F.Cu at (227.3, 77.6)
- added D207: grün, LED_THT:LED_D5.0mm, F.Cu at (234.8, 77.6)
- added D208: rot, LED_THT:LED_Rectangular_W3.0mm_H2.0mm, F.Cu at (204.0, 90.7)
- added D209: rot, LED_THT:LED_Rectangular_W3.0mm_H2.0mm, F.Cu at (204.0, 94.5)
- added D210: rot, LED_THT:LED_Rectangular_W3.0mm_H2.0mm, F.Cu at (204.0, 98.2)
- added D211: rot, LED_THT:LED_Rectangular_W3.0mm_H2.0mm, F.Cu at (204.0, 102.0)
- added D212: rot, LED_THT:LED_Rectangular_W3.0mm_H2.0mm, F.Cu at (204.0, 105.7)
- added D213: rot, LED_THT:LED_Rectangular_W3.0mm_H2.0mm, F.Cu at (204.0, 109.5)
- added D301: wasserblau, LED_SMD:LED_0603_1608Metric, F.Cu at (268.2, 46.9)
- added D302: wasserblau, LED_SMD:LED_0603_1608Metric, F.Cu at (268.2, 49.5)
- added D401: wasserblau, LED_SMD:LED_0603_1608Metric, F.Cu at (275.1, 86.4)
- added D402: 1N4148, Diode_SMD:D_MiniMELF, F.Cu at (251.2, 97.7)
- added D403: wasserblau, LED_SMD:LED_0603_1608Metric, F.Cu at (275.1, 89.0)
- added D404: 1N4148, Diode_SMD:D_MiniMELF, F.Cu at (251.2, 101.1)
- added D405: wasserblau, LED_SMD:LED_0603_1608Metric, F.Cu at (275.1, 91.6)
- added D406: wasserblau, LED_SMD:LED_0603_1608Metric, F.Cu at (275.1, 94.2)
- added F103: Fuse, Resistor_SMD:R_1210_3225Metric, F.Cu at (209.8, 57.8)
- added F104: Fuse, Resistor_SMD:R_1210_3225Metric, F.Cu at (209.8, 62.0)
- added J110: DS18B20, Connector_JST:JST_XH_B3B-XH-AM_1x03_P2.50mm_Vertical, F.Cu at (235.2, 55.7)
- added J111: BMP280, Connector_PinHeader_2.54mm:PinHeader_1x06_P2.54mm_Vertical, F.Cu at (204.7, 50.2)
- added J113: RS485-mini-1, Connector_JST:JST_XH_B2B-XH-AM_1x02_P2.50mm_Vertical, F.Cu at (210.5, 51.2)
- added J114: AVR-ISP-6, Connector_IDC:IDC-Header_2x03_P2.54mm_Vertical, F.Cu at (223.6, 33.9)
- added JP101: 24V_ext, Connector_PinHeader_2.54mm:PinHeader_1x02_P2.54mm_Vertical, F.Cu at (220.7, 47.5)
- added JP102: 5V_ext, Connector_PinHeader_2.54mm:PinHeader_1x02_P2.54mm_Vertical, F.Cu at (225.4, 47.5)
- added JP103: WP_OFF, Connector_PinHeader_2.54mm:PinHeader_1x02_P2.54mm_Vertical, F.Cu at (230.0, 47.5)
- added K401: V23040, board:V23040, F.Cu at (259.0, 79.4)
- added K402: V23040, board:V23040, F.Cu at (259.0, 90.5)
- added L301: 15uH, Inductor_SMD:L_Bourns-SRN4018, F.Cu at (263.1, 48.4)
- added NT101: Massesternpunkt, NetTie:NetTie-2_SMD_Pad0.5mm, F.Cu at (208.5, 70.7)
- added Q1: BC817, Package_TO_SOT_SMD:SOT-23, F.Cu at (220.8, 54.6)
- added Q2: BC817, Package_TO_SOT_SMD:SOT-23, F.Cu at (220.8, 59.0)
- added Q201: BC807, Package_TO_SOT_SMD:SOT-23, F.Cu at (242.0, 83.6)
- added Q401: BC817, Package_TO_SOT_SMD:SOT-23, F.Cu at (275.5, 97.7)
- added Q402: BC817, Package_TO_SOT_SMD:SOT-23, F.Cu at (275.5, 102.2)
- added R125: 10k, Resistor_SMD:R_0603_1608Metric, F.Cu at (208.4, 46.6)
- added R126: 15R, Resistor_SMD:R_1206_3216Metric, F.Cu at (226.1, 66.9)
- added R127: 100k, Resistor_SMD:R_0603_1608Metric, F.Cu at (212.4, 29.1)
- added R128: 100k, Resistor_SMD:R_0603_1608Metric, F.Cu at (212.4, 31.6)
- added R129: 4,7k, Resistor_SMD:R_0603_1608Metric, F.Cu at (212.4, 34.1)
- added R130: 10k, Resistor_SMD:R_0603_1608Metric, F.Cu at (212.4, 36.6)
- added R131: tbd, Resistor_SMD:R_0603_1608Metric, F.Cu at (212.4, 39.1)
- added R132: tbd, Resistor_SMD:R_0603_1608Metric, F.Cu at (212.4, 41.6)
- added R133: tbd, Resistor_SMD:R_0603_1608Metric, F.Cu at (212.4, 44.1)
- added R134: tbd, Resistor_SMD:R_0603_1608Metric, F.Cu at (212.4, 46.6)
- added R135: 3,3k, Resistor_SMD:R_0603_1608Metric, F.Cu at (216.4, 29.1)
- added R136: 3,3k, Resistor_SMD:R_0603_1608Metric, F.Cu at (216.4, 31.6)
- added R137: 33k, Resistor_SMD:R_0603_1608Metric, F.Cu at (216.4, 34.1)
- added R138: NC, Resistor_SMD:R_1206_3216Metric, F.Cu at (226.1, 70.2)
- added R139: 1k, Resistor_SMD:R_0603_1608Metric, F.Cu at (216.4, 36.6)
- added R301: 1k, Resistor_SMD:R_0603_1608Metric, F.Cu at (252.4, 34.1)
- added R302: 510k, Resistor_SMD:R_0603_1608Metric, F.Cu at (252.4, 36.6)
- added R303: 49,9, Resistor_SMD:R_0603_1608Metric, F.Cu at (252.4, 39.1)
- added R304: 100k, Resistor_SMD:R_0603_1608Metric, F.Cu at (252.4, 41.6)
- added R305: 10k, Resistor_SMD:R_0603_1608Metric, F.Cu at (252.4, 44.1)
- added R306: 2,2k, Resistor_SMD:R_0603_1608Metric, F.Cu at (252.4, 46.6)
- added R307: 3,3k, Resistor_SMD:R_0603_1608Metric, F.Cu at (252.4, 49.1)
- added R401: 2,2k, Resistor_SMD:R_0603_1608Metric, F.Cu at (271.1, 86.4)
- added R402: 10k, Resistor_SMD:R_0603_1608Metric, F.Cu at (271.1, 88.9)
- added R403: 220R, Resistor_SMD:R_0603_1608Metric, F.Cu at (271.1, 91.4)
- added R404: 2,2k, Resistor_SMD:R_0603_1608Metric, F.Cu at (271.1, 93.9)
- added R405: 10k, Resistor_SMD:R_0603_1608Metric, F.Cu at (271.1, 96.4)
- added R406: 220R, Resistor_SMD:R_0603_1608Metric, F.Cu at (271.1, 98.9)
- added RN101: 56k, Resistor_SMD:R_Array_Convex_4x1206, F.Cu at (235.1, 48.5)
- added RN102: 56k, Resistor_SMD:R_Array_Convex_4x1206, F.Cu at (240.5, 48.5)
- added RN201: 220R, Resistor_SMD:R_Array_Convex_4x1206, F.Cu at (211.0, 84.7)
- added RN202: 220R, Resistor_SMD:R_Array_Convex_4x1206, F.Cu at (216.4, 84.7)
- added RN203: 220R, Resistor_SMD:R_Array_Convex_4x1206, F.Cu at (221.9, 84.7)
- added RN204: 220R, Resistor_SMD:R_Array_Convex_4x1206, F.Cu at (227.4, 84.7)
- added RN205: 220R, Resistor_SMD:R_Array_Convex_4x1206, F.Cu at (232.8, 84.7)
- added RN206: 220R, Resistor_SMD:R_Array_Convex_4x1206, F.Cu at (211.0, 91.5)
- added RN207: 220R, Resistor_SMD:R_Array_Convex_4x1206, F.Cu at (216.4, 91.5)
- added RN208: 220R, Resistor_SMD:R_Array_Convex_4x1206, F.Cu at (221.9, 91.5)
- added RN209: 220R, Resistor_SMD:R_Array_Convex_4x1206, F.Cu at (227.4, 91.5)
- added RN210: 220R, Resistor_SMD:R_Array_Convex_4x1206, F.Cu at (232.8, 91.5)
- added RN211: 220R, Resistor_SMD:R_Array_Convex_4x1206, F.Cu at (211.0, 98.2)
- added RN212: 220R, Resistor_SMD:R_Array_Convex_4x1206, F.Cu at (216.4, 98.2)
- added RN213: 220R, Resistor_SMD:R_Array_Convex_4x1206, F.Cu at (221.9, 98.2)
- added TP101: Pin_7, TestPoint:TestPoint_Keystone_5005-5009_Compact, F.Cu at (245.9, 62.7)
- added TP102: Pin_8, TestPoint:TestPoint_Keystone_5005-5009_Compact, F.Cu at (245.9, 67.7)
- added U103: ATmega8A-A, Package_QFP:TQFP-32_7x7mm_P0.8mm, F.Cu at (237.6, 66.0)
- added U104: REF3040, Package_TO_SOT_SMD:SOT-23, F.Cu at (220.8, 63.5)
- added U105: 74HC165, Package_SO:SOIC-16_3.9x9.9mm_P1.27mm, F.Cu at (234.6, 33.5)
- added U106: 74HC595, Package_SO:SOIC-16_3.9x9.9mm_P1.27mm, F.Cu at (243.0, 33.5)
- added U107: SN75176AD, Package_SO:SOIC-8_3.9x4.9mm_P1.27mm, F.Cu at (227.5, 55.6)
- added U108: CAT24M01W, Package_SO:SOIC-8_3.9x4.9mm_P1.27mm, F.Cu at (227.5, 62.0)
- added U209: 74HC595, Package_SO:SOIC-16_3.9x9.9mm_P1.27mm, F.Cu at (233.3, 107.3)
- added U210: 5161BK, Display_7Segment:D1X8K, F.Cu at (211.1, 103.6)
- added U211: 74HC595, Package_SO:SOIC-16_3.9x9.9mm_P1.27mm, F.Cu at (241.7, 107.3)
- added U301: TPS54202DDC, Package_TO_SOT_SMD:SOT-23-6, F.Cu at (257.0, 46.8)
- added U302: AP1117-33, Package_TO_SOT_SMD:SOT-223-3_TabPin2, F.Cu at (265.0, 31.9)
- added U401: CPC1002N, Package_SO:SOP-4_3.8x4.1mm_P2.54mm, F.Cu at (273.3, 76.6)
- added U402: CPC1002N, Package_SO:SOP-4_3.8x4.1mm_P2.54mm, F.Cu at (273.3, 82.3)
- added Y101: 16MHz, Crystal:Resonator_SMD_Murata_CSTxExxV-3Pin_3.0x1.1mm, F.Cu at (245.8, 46.9)
- C101: value 1µ 16V -> paar nF; footprint Capacitor_SMD:C_0805_2012Metric -> Capacitor_SMD:C_0603_1608Metric
- C108, C109: value 100n -> 1u
- C110, C111: value 100n -> 470n
- D101: value grün -> SP0502BAHT; footprint LED_SMD:LED_0603_1608Metric -> Package_TO_SOT_SMD:SOT-23
- D106: value grün -> SM6T30A; footprint LED_SMD:LED_0603_1608Metric -> Diode_SMD:D_SMB
- J101: value Conn_01x02 -> 24V in; footprint TerminalBlock:TerminalBlock_bornier-4_P5.08mm -> Connector_JST:JST_XH_B2B-XH-A_1x02_P2.50mm_Vertical; moved to F.Cu
- J103: value RJ45 -> RS485-mini-1; footprint Sven:RJ45_Amphenol_54602_mod -> Connector_JST:JST_XH_B2B-XH-AM_1x02_P2.50mm_Vertical
- R101: value 470 -> 15R; footprint Resistor_SMD:R_0603_1608Metric -> Resistor_SMD:R_1206_3216Metric
- R102: value 10k -> 1k
- R103, R104: value 10k -> 24k 1%
- R109, R115: value 10k -> 20k 1%
- R110, R114: value 10k -> 33k 1%
- R111: value 10k -> 33k
- R112: footprint Resistor_SMD:R_0603_1608Metric -> Resistor_SMD:R_1206_3216Metric
- R113: value 470 -> 1k
- R201: value R -> 10k*; footprint Resistor_SMD:R_0805_2012Metric -> Resistor_SMD:R_0603_1608Metric
- R202, R205, R206: value R -> 10k; footprint Resistor_SMD:R_0805_2012Metric -> Resistor_SMD:R_0603_1608Metric
- R203, R204: value R -> 220R; footprint Resistor_SMD:R_0805_2012Metric -> Resistor_SMD:R_0603_1608Metric
- U201, U203, U205: value KCSA02-106 -> 8106BS; footprint Display_7Segment:7SEGMENT-LED__HDSM531_HDSM533_SMD -> board:8106BS
- U207: value KCSA02-106 -> 5161BK; footprint Display_7Segment:7SEGMENT-LED__HDSM531_HDSM533_SMD -> Display_7Segment:D1X8K
- moved J103 238.8 mm to (273.3, 151.1), turned to 90 degrees
- moved F102 223.6 mm to (275.6, 130.3), turned to 90 degrees
- moved D105 222.9 mm to (270.5, 158.7), turned to 90 degrees
- moved D106 214.6 mm to (276.0, 158.7), turned to 90 degrees
- moved R104 213.7 mm to (268.4, 139.1), turned to 90 degrees
- moved D101 213.7 mm to (278.1, 125.0), turned to 90 degrees
- moved R111 212.9 mm to (276.0, 139.1), turned to 90 degrees
- moved R114 212.5 mm to (265.9, 135.1), turned to 90 degrees
- moved R102 212.0 mm to (263.4, 139.1), turned to 90 degrees
- moved R115 210.7 mm to (268.4, 135.1), turned to 90 degrees
- moved R109 210.7 mm to (270.9, 139.1), turned to 90 degrees
- moved R110 209.2 mm to (273.5, 139.1), turned to 90 degrees
- moved R101 207.7 mm to (271.0, 124.7), turned to 90 degrees
- moved R103 203.2 mm to (265.9, 139.1), turned to 90 degrees
- moved R112 194.1 mm to (274.2, 124.7), turned to 90 degrees
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Connections:
- net /7SegClk renamed /SCK_Schieber_Takt
- net /Magnetron_ADC renamed /ADC6_Messröhre 1 Signal
- C101 pad 2: +5V -> /DS18B20_Anschluss
- C108 pad 1: /Pirani_Ident -> /ADC1_ID_2
- C109 pad 1: /Pirani_ADC -> /ADC0_ID_1
- C110 pad 2: GND -> GNDA
- C111 pad 1: /Magnetron_Setpoint_ADC -> /ADC7_Messröhre 2 Signal
- C111 pad 2: GND -> GNDA
- D101 pad 1: Net-(D101-Pad1) -> /RS485_A
- D101 pad 2: Net-(D101-Pad2) -> /RS485_B
- D103 pad 1: /24_Ext -> +24V
- D103 pad 2: GNDPWR -> GND
- D105 pad 1: Net-(D105-Pad1) -> +5V
- D105 pad 2: /Magnetron_Trip -> /DS18B20_Anschluss
- D106 pad 1: Net-(D106-Pad1) -> /R2_Switch_Pulldown
- D106 pad 2: Net-(D106-Pad2) -> GND
- F102 pad 1: GND -> +24V
- F102 pad 2: GNDPWR -> Net-(J101-Pin_1)
- J101 pad 1: /24_Ext -> Net-(J101-Pin_1)
- J101 pad 2: GNDPWR -> GND
- J103 pad 1: /Pirani_Ident -> /RS485_B
- J103 pad 2: Net-(J103-Pad2) -> /RS485_A
- R101 pad 1: +5V -> Net-(U104-IN)
- R101 pad 2: Net-(D101-Pad2) -> +5V
- R102 pad 1: /Pirani_ADC -> Net-(U105-Q7)
- R102 pad 2: GND -> /MISO_Schieber_Daten_In
- R103 pad 2: GND -> GNDA
- R104 pad 1: /Magnetron_Setpoint_ADC -> /ADC7_Messröhre 2 Signal
- R104 pad 2: GND -> GNDA
- R110 pad 2: GND -> GNDA
- R111 pad 1: /Magnetron_Trip -> /ADC0_ID_1
- R112 pad 2: Net-(J104-Pad7) -> /R1_Switch_Pulldown
- R113 pad 1: +5V -> /R1_MagEn
- R113 pad 2: Net-(D106-Pad2) -> Net-(Q1-B)
- R114 pad 1: Net-(J104-Pad8) -> /ADC7_Messröhre 2 Signal
- R114 pad 2: /Magnetron_Setpoint_ADC -> GNDA
- R115 pad 1: /Magnetron_Setpoint_ADC -> Net-(C129-Pad1)
- R115 pad 2: GND -> /ADC7_Messröhre 2 Signal
- R201 pad 1: Net-(R201-Pad1) -> +5V
- R201 pad 2: Net-(R201-Pad2) -> /OC1A_Dimmer
- R202 pad 1: Net-(R202-Pad1) -> /OC1A_Dimmer
- R202 pad 2: Net-(R202-Pad2) -> Net-(Q201-B)
- R203 pad 1: Net-(R203-Pad1) -> Net-(D202-A)
- R203 pad 2: Net-(R203-Pad2) -> Net-(Q201-C)
- R204 pad 1: Net-(R204-Pad1) -> Net-(D201-A)
- R204 pad 2: Net-(R204-Pad2) -> Net-(Q201-C)
- R205 pad 1: Net-(R205-Pad1) -> /OC1A_Dimmer
- R205 pad 2: Net-(R205-Pad2) -> GND
- R206 pad 1: Net-(R206-Pad1) -> /SS_Schieber_Latch
- R206 pad 2: Net-(R206-Pad2) -> GND
- U201 pad 1: Net-(R205-Pad2) -> +5V
- U201 pad 2: Net-(R204-Pad2) -> Net-(RN202-R1.2)
- U201 pad 3: +5V -> Net-(RN201-R4.2)
- U201 pad 4: Net-(R203-Pad2) -> Net-(RN201-R3.2)
- U201 pad 5: Net-(R208-Pad2) -> +5V
- U201 pad 6: Net-(R202-Pad2) -> Net-(RN201-R2.2)
- U201 pad 7: Net-(R201-Pad2) -> Net-(RN201-R1.2)
- U201 pad 8: +5V -> Net-(RN202-R4.2)
- U201 pad 9: Net-(R206-Pad2) -> Net-(RN202-R2.2)
- U202 pad 1: Net-(R202-Pad1) -> Net-(RN201-R2.1)
- U202 pad 12: /7SegEN -> /SS_Schieber_Latch
- U202 pad 13: GND -> /OC1A_Dimmer
- U202 pad 14: /7SegData -> /MOSI_Schieber_Daten_Out
- U202 pad 15: Net-(R201-Pad1) -> Net-(RN201-R1.1)
- U202 pad 2: Net-(R203-Pad1) -> Net-(RN201-R3.1)
- U202 pad 3: Net-(R204-Pad1) -> Net-(RN201-R4.1)
- U202 pad 4: Net-(R205-Pad1) -> Net-(RN202-R1.1)
- U202 pad 5: Net-(R206-Pad1) -> Net-(RN202-R2.1)
- U203 pad 1: Net-(R213-Pad2) -> +5V
- U203 pad 3: +5V -> Net-(RN203-R4.2)
- U203 pad 5: Net-(R216-Pad2) -> +5V
- U203 pad 8: +5V -> Net-(RN204-R4.2)
- U204 pad 12: /7SegEN -> /SS_Schieber_Latch
- U204 pad 13: GND -> /OC1A_Dimmer
- U205 pad 1: Net-(R221-Pad2) -> +5V
- U205 pad 3: +5V -> Net-(RN205-R4.2)
- U205 pad 5: Net-(R224-Pad2) -> +5V
- U205 pad 8: +5V -> Net-(RN206-R4.2)
- U206 pad 12: /7SegEN -> /SS_Schieber_Latch
- U206 pad 13: GND -> /OC1A_Dimmer
- U208 pad 12: /7SegEN -> /SS_Schieber_Latch
- U208 pad 13: GND -> /OC1A_Dimmer
- U208 pad 9: unconnected-(U208-Pad9) -> Net-(U208-QH')
Routing:
- net +5V: track 301.2 -> 0.00 mm, vias 20 -> 0
- net /Tacho: track 125.0 -> 0.00 mm, vias 4 -> 0
- net /7SegEN: track 121.8 -> 0.00 mm
- net /SCK_Schieber_Takt: track 120.3 -> 0.00 mm
- net /TX_2: track 112.2 -> 0.00 mm, vias 4 -> 0
- net /RX_2: track 107.4 -> 0.00 mm, vias 4 -> 0
- net /Pirani_Ident: track 95.0 -> 0.00 mm, vias 1 -> 0
- net GND: track 89.4 -> 0.00 mm, vias 17 -> 0
- net /EnableAll: track 79.2 -> 0.00 mm, vias 1 -> 0
- net /Magnetron_Enable: track 73.2 -> 0.00 mm, vias 1 -> 0
- net /Main_ON: track 72.2 -> 0.00 mm, vias 5 -> 0
- net /Pirani_ADC: track 72.1 -> 0.00 mm, vias 3 -> 0
- net +24V: track 71.8 -> 0.00 mm, vias 1 -> 0
- net /Magnetron_Setpoint_ADC: track 69.4 -> 0.00 mm, vias 1 -> 0
- net /RS232_TX: track 68.9 -> 0.00 mm, vias 1 -> 0
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- removed copper zone on B.Cu, net /24_Ext
- removed copper zone on B.Cu, net GND
- removed copper zone on F.Cu, net GND
- removed copper zone on F.Cu, net GNDPWR

Commit message: kleine änderungen
Parts:
- added C102: 100n, Capacitor_SMD:C_0603_1608Metric, F.Cu at (259.2, 116.5)
- added C103: 100n, Capacitor_SMD:C_0603_1608Metric, F.Cu at (259.2, 119.0)
- added C104: 100n, Capacitor_SMD:C_0603_1608Metric, F.Cu at (259.2, 121.5)
- added R105: 15R, Resistor_SMD:R_0603_1608Metric, F.Cu at (259.2, 124.0)
- added R106: 15R, Resistor_SMD:R_0603_1608Metric, F.Cu at (259.2, 126.5)
- added R107: 15R, Resistor_SMD:R_0603_1608Metric, F.Cu at (259.2, 129.0)
- added SW101: SW_Omron_B3FS, Button_Switch_THT:SW_PUSH-12mm, F.Cu at (242.4, 119.5)
- added SW102: SW_Omron_B3FS, Button_Switch_THT:SW_PUSH-12mm, F.Cu at (242.4, 133.0)
- added SW104: SW_Omron_B3FS, Button_Switch_THT:SW_PUSH-12mm, F.Cu at (242.4, 146.6)
- C127, C128: value 100p -> 100n
- R131, R132: value tbd -> 4,7k
- R133: value tbd -> 1,8k
- R134: value tbd -> 33k
- RN201, RN202, RN203, RN204, RN205, RN206, RN207, RN208, RN209, RN210, RN211, RN213, U202, U204, U206, U208, U209, U211: moved to B.Cu
- moved D212 149.2 mm to (56.5, 84.0)
- moved U211 148.7 mm to (99.3, 64.6), turned to 180 degrees
- moved D210 143.5 mm to (61.5, 81.5), turned to 90 degrees
- moved D211 143.2 mm to (61.5, 89.0), turned to 90 degrees
- moved D213 142.3 mm to (64.0, 84.0)
- moved RN202 134.4 mm to (82.0, 86.0)
- moved U205 130.6 mm to (115.9, 95.5)
- moved U203 130.1 mm to (95.5, 95.5)
- moved U201 129.7 mm to (74.9, 95.5)
- moved RN201 129.1 mm to (82.0, 80.0)
- moved RN204 124.4 mm to (103.0, 86.0)
- moved U202 121.3 mm to (75.5, 83.8), turned to 180 degrees
- moved RN203 119.0 mm to (103.0, 80.0)
- moved RN213 118.7 mm to (108.8, 62.0), turned to -90 degrees
- moved RN205 109.4 mm to (123.5, 80.0)
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Connections:
- U201 pad 10: Net-(RN202-R3.2) -> Net-(RN202-R2.2)
- U201 pad 2: Net-(RN202-R1.2) -> Net-(RN202-R4.2)
- U201 pad 3: Net-(RN201-R4.2) -> Net-(RN201-R1.2)
- U201 pad 4: Net-(RN201-R3.2) -> Net-(RN201-R2.2)
- U201 pad 6: Net-(RN201-R2.2) -> Net-(RN201-R3.2)
- U201 pad 7: Net-(RN201-R1.2) -> Net-(RN201-R4.2)
- U201 pad 8: Net-(RN202-R4.2) -> Net-(RN202-R1.2)
- U201 pad 9: Net-(RN202-R2.2) -> Net-(RN202-R3.2)
- U202 pad 1: Net-(RN201-R2.1) -> Net-(RN201-R3.1)
- U202 pad 15: Net-(RN201-R1.1) -> Net-(RN201-R4.1)
- U202 pad 2: Net-(RN201-R3.1) -> Net-(RN201-R2.1)
- U202 pad 3: Net-(RN201-R4.1) -> Net-(RN201-R1.1)
- U202 pad 4: Net-(RN202-R1.1) -> Net-(RN202-R4.1)
- U202 pad 5: Net-(RN202-R2.1) -> Net-(RN202-R3.1)
- U202 pad 6: Net-(RN202-R3.1) -> Net-(RN202-R2.1)
- U202 pad 7: Net-(RN202-R4.1) -> Net-(RN202-R1.1)
- U203 pad 10: Net-(RN204-R3.2) -> Net-(RN204-R2.2)
- U203 pad 2: Net-(RN204-R1.2) -> Net-(RN204-R4.2)
- U203 pad 3: Net-(RN203-R4.2) -> Net-(RN203-R1.2)
- U203 pad 4: Net-(RN203-R3.2) -> Net-(RN203-R2.2)
- U203 pad 6: Net-(RN203-R2.2) -> Net-(RN203-R3.2)
- U203 pad 7: Net-(RN203-R1.2) -> Net-(RN203-R4.2)
- U203 pad 8: Net-(RN204-R4.2) -> Net-(RN204-R1.2)
- U203 pad 9: Net-(RN204-R2.2) -> Net-(RN204-R3.2)
- U204 pad 1: Net-(RN203-R2.1) -> Net-(RN203-R3.1)
- U204 pad 15: Net-(RN203-R1.1) -> Net-(RN203-R4.1)
- U204 pad 2: Net-(RN203-R3.1) -> Net-(RN203-R2.1)
- U204 pad 3: Net-(RN203-R4.1) -> Net-(RN203-R1.1)
- U204 pad 4: Net-(RN204-R1.1) -> Net-(RN204-R4.1)
- U204 pad 5: Net-(RN204-R2.1) -> Net-(RN204-R3.1)
- U204 pad 6: Net-(RN204-R3.1) -> Net-(RN204-R2.1)
- U204 pad 7: Net-(RN204-R4.1) -> Net-(RN204-R1.1)
- U205 pad 10: Net-(RN206-R3.2) -> Net-(RN206-R2.2)
- U205 pad 2: Net-(RN206-R1.2) -> Net-(RN206-R4.2)
- U205 pad 3: Net-(RN205-R4.2) -> Net-(RN205-R1.2)
- U205 pad 4: Net-(RN205-R3.2) -> Net-(RN205-R2.2)
- U205 pad 6: Net-(RN205-R2.2) -> Net-(RN205-R3.2)
- U205 pad 7: Net-(RN205-R1.2) -> Net-(RN205-R4.2)
- U205 pad 8: Net-(RN206-R4.2) -> Net-(RN206-R1.2)
- U205 pad 9: Net-(RN206-R2.2) -> Net-(RN206-R3.2)
- U206 pad 1: Net-(RN205-R2.1) -> Net-(RN205-R3.1)
- U206 pad 15: Net-(RN205-R1.1) -> Net-(RN205-R4.1)
- U206 pad 2: Net-(RN205-R3.1) -> Net-(RN205-R2.1)
- U206 pad 3: Net-(RN205-R4.1) -> Net-(RN205-R1.1)
- U206 pad 4: Net-(RN206-R1.1) -> Net-(RN206-R4.1)
- U206 pad 5: Net-(RN206-R2.1) -> Net-(RN206-R3.1)
- U206 pad 6: Net-(RN206-R3.1) -> Net-(RN206-R2.1)
- U206 pad 7: Net-(RN206-R4.1) -> Net-(RN206-R1.1)
- U207 pad 1: Net-(RN208-R1.2) -> Net-(RN208-R4.2)
- U207 pad 10: Net-(RN208-R3.2) -> Net-(RN208-R2.2)
- U207 pad 2: Net-(RN207-R4.2) -> Net-(RN207-R1.2)
- U207 pad 4: Net-(RN207-R3.2) -> Net-(RN207-R2.2)
- U207 pad 5: Net-(RN208-R4.2) -> Net-(RN208-R1.2)
- U207 pad 6: Net-(RN207-R2.2) -> Net-(RN207-R3.2)
- U207 pad 7: Net-(RN207-R1.2) -> Net-(RN207-R4.2)
- U207 pad 9: Net-(RN208-R2.2) -> Net-(RN208-R3.2)
- U208 pad 1: Net-(RN207-R2.1) -> Net-(RN207-R3.1)
- U208 pad 15: Net-(RN207-R1.1) -> Net-(RN207-R4.1)
- U208 pad 2: Net-(RN207-R3.1) -> Net-(RN207-R2.1)
- U208 pad 3: Net-(RN207-R4.1) -> Net-(RN207-R1.1)
- U208 pad 4: Net-(RN208-R1.1) -> Net-(RN208-R4.1)
- U208 pad 5: Net-(RN208-R2.1) -> Net-(RN208-R3.1)
- U208 pad 6: Net-(RN208-R3.1) -> Net-(RN208-R2.1)
- U208 pad 7: Net-(RN208-R4.1) -> Net-(RN208-R1.1)
- U209 pad 1: Net-(RN209-R2.1) -> Net-(RN209-R3.1)
- U209 pad 15: Net-(RN209-R1.1) -> Net-(RN209-R4.1)
- U209 pad 2: Net-(RN209-R3.1) -> Net-(RN209-R2.1)
- U209 pad 3: Net-(RN209-R4.1) -> Net-(RN209-R1.1)
- U209 pad 4: Net-(RN210-R1.1) -> Net-(RN210-R4.1)
- U209 pad 5: Net-(RN210-R2.1) -> Net-(RN210-R3.1)
- U209 pad 6: Net-(RN210-R3.1) -> Net-(RN210-R2.1)
- U209 pad 7: Net-(RN210-R4.1) -> Net-(RN210-R1.1)
- U210 pad 1: Net-(RN210-R1.2) -> Net-(RN210-R4.2)
- U210 pad 10: Net-(RN210-R3.2) -> Net-(RN210-R2.2)
- U210 pad 2: Net-(RN209-R4.2) -> Net-(RN209-R1.2)
- U210 pad 4: Net-(RN209-R3.2) -> Net-(RN209-R2.2)
- U210 pad 5: Net-(RN210-R4.2) -> Net-(RN210-R1.2)
- U210 pad 6: Net-(RN209-R2.2) -> Net-(RN209-R3.2)
- U210 pad 7: Net-(RN209-R1.2) -> Net-(RN209-R4.2)
- U210 pad 9: Net-(RN210-R2.2) -> Net-(RN210-R3.2)

Commit message: Layout weitergemacht, RJ45 Buchsen fehlen noch komplett
Parts:
- removed D104: SD05_SOD323, Diode_SMD:D_SOD-323
- removed REF**: STS, Sven:STS
- added D1: SMF5.0A, Diode_SMD:D_SOD-123F, F.Cu at (253.8, 56.6)
- added D2: SMF5.0A, Diode_SMD:D_SOD-123F, F.Cu at (253.8, 60.0)
- added D3: SMF5.0A, Diode_SMD:D_SOD-123F, F.Cu at (253.8, 63.3)
- added SW103: SW_DIP_x08, Button_Switch_THT:SW_DIP_SPSTx08_Slide_9.78x22.5mm_W7.62mm_P2.54mm, F.Cu at (188.4, 81.5)
- C102, C103, C104, R105, R106, R107, RN101, RN102, RN212, U105: moved to B.Cu
- R111, R137: value 33k -> 18k
- moved D207 189.8 mm to (47.5, 57.5)
- moved D206 180.0 mm to (47.5, 65.0)
- moved C104 171.4 mm to (88.0, 112.8), turned to 90 degrees
- moved R105 171.4 mm to (88.0, 116.2), turned to 90 degrees
- moved SW101 170.0 mm to (72.5, 112.5)
- moved D205 162.8 mm to (47.5, 100.0)
- moved RN212 160.4 mm to (71.5, 61.8), turned to 180 degrees
- moved D204 154.0 mm to (47.5, 107.5)
- moved D203 145.6 mm to (47.5, 115.0)
- moved SW102 143.9 mm to (100.0, 112.5)
- moved R106 143.5 mm to (116.0, 116.2), turned to 90 degrees
- moved C103 143.3 mm to (116.0, 112.8), turned to 90 degrees
- moved SW104 119.8 mm to (127.5, 112.5)
- moved R107 115.9 mm to (144.0, 116.2), turned to 90 degrees
- moved C102 115.2 mm to (144.0, 112.8), turned to -90 degrees
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Other:
- board outline removed
- board text added: "Absolutdruck"
- board text added: "Atmosphäre"
- board text added: "Eingang 1"
- board text added: "Eingang 2"
- board text added: "Eurokartenmaß"
- board text added: "Relativdruck"
- board text removed: "(C)2021 S.T.Schneider"
- board text removed: "24V"
- board text removed: "24V GND"
- board text removed: "AIM-X"
- board text removed: "Bridge for RX/TX_0"
- board text removed: "Bridge for direct RX/TX Open for RS232"
- board text removed: "Edwards Magnetron"
- board text removed: "Edwards Turbo"
- board text removed: "Fan"
- board text removed: "GND"
- board text removed: "High-Vacuum-Shield"
- board text removed: "Jump_Serial"
- board text removed: "OFF"
- board text removed: "ON"
- board text removed: "Pfeiffer Pirani"
- board text removed: "Pirani"
- board text removed: "Pirani 1E+3 1E-3 Magnetron 1E-2 1E-9"
- board text removed: "RX TX"
- board text removed: "Rev: 1"
- board text removed: "Switch_Start"
- board text removed: "TX RX"
- board text removed: "Tacho"

Commit message: Stecker fertig ausgewählt und Layout etwa 60% fertig
Parts:
- added H101: MountingHole, MountingHole:MountingHole_3.2mm_M3_DIN965, F.Cu at (45.0, 82.5)
- added H102: MountingHole, MountingHole:MountingHole_3.2mm_M3_DIN965, F.Cu at (45.0, 145.0)
- added H103: MountingHole, MountingHole:MountingHole_3.2mm_M3_DIN965, F.Cu at (195.0, 145.0)
- added H104: MountingHole, MountingHole:MountingHole_3.2mm_M3_DIN965, F.Cu at (195.0, 60.0)
- added J104: RJ45, board:RJ45_Amphenol_54602_mod, B.Cu at (52.8, 122.3)
- added J108: RJ45, board:RJ45_Amphenol_54602_mod, B.Cu at (187.2, 115.2)
- added J109: RJ45, board:RJ45_Amphenol_54602_mod, B.Cu at (187.2, 133.2)
- added J112: RJ45, board:RJ45_Amphenol_54602_mod, B.Cu at (52.8, 104.3)
- added J401: Conn_01x03, Connector_Wago:Wago_734-133_1x03_P3.50mm_Vertical, B.Cu at (72.5, 129.0)
- added J402: Conn_01x03, Connector_Wago:Wago_734-133_1x03_P3.50mm_Vertical, B.Cu at (72.5, 144.7)
- added J403: Conn_01x02, Connector_Wago:Wago_734-132_1x02_P3.50mm_Vertical, B.Cu at (111.7, 143.9)
- added J404: Conn_01x02, Connector_Wago:Wago_734-132_1x02_P3.50mm_Vertical, B.Cu at (124.3, 144.0)
- C101, C108, C109, C110, C111, C114, C115, C116, C117, C118, C119, C120, C121, C122, C123, C124, C125, C126, C127, C128, C129, C130, C201, C202, C203, C204, C205, C206, C301, C302, C303, C304, C305, C306, C307, C308, D1, D101, D102, D103, D105, D106, D2, D3, D301, D302, D401, D402, D403, D404, D405, D406, F102, F103, F104, J101, J103, J110, J111, J113, J114, JP103, K401, K402, L301, NT101, Q1, Q2, Q201, Q401, Q402, R101, R102, R103, R104, R109, R110, R111, R112, R113, R114, R115, R125, R126, R127, R128, R129, R130, R131, R132, R133, R134, R135, R136, R137, R138, R139, R201, R202, R203, R204, R205, R206, R302, R303, R304, R305, R307, R401, R402, R403, R404, R405, R406, SW103, TP101, TP102, U103, U104, U106, U107, U108, U301, U302, U401, U402, Y101: moved to B.Cu
- R301: value 1k -> 4,7k; moved to B.Cu
- R306: value 2,2k -> 10k; moved to B.Cu
- moved D106 236.4 mm to (49.0, 93.0), turned to 180 degrees
- moved R112 222.1 mm to (52.5, 137.5), turned to 180 degrees
- moved R111 219.2 mm to (57.6, 119.8), turned to 0 degrees
- moved C111 215.5 mm to (63.4, 107.6)
- moved C108 215.2 mm to (57.6, 100.2), turned to 0 degrees
- moved C109 214.8 mm to (57.6, 118.2), turned to 0 degrees
- moved R109 213.7 mm to (57.6, 126.4), turned to 0 degrees
- moved R115 212.6 mm to (57.5, 108.5), turned to 0 degrees
- moved R110 212.1 mm to (61.8, 125.6)
- moved C110 210.8 mm to (63.4, 125.6)
- moved R104 210.6 mm to (60.2, 107.6)
- moved R113 208.4 mm to (55.0, 134.0)
- moved R103 206.2 mm to (60.2, 125.6)
- moved R114 206.0 mm to (61.8, 107.6)
- moved D2 205.2 mm to (58.2, 122.0)
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Connections:
- C117 pad 2: GND -> GNDA
- C121 pad 2: GND -> GNDA
- RN212 pad 5: /7-Segment/In3aktiv -> /7-Segment/AnzeigeRelativdruck
- RN212 pad 6: /7-Segment/In2aktiv -> /7-Segment/In1aktiv
- RN212 pad 7: /7-Segment/In1aktiv -> /7-Segment/In2aktiv
- RN212 pad 8: /7-Segment/AnzeigeRelativdruck -> /7-Segment/In3aktiv
- U103 pad 25: /ADC2_5V_Versorgung -> /ADC3_24V_Versorgung
- U103 pad 26: /ADC3_24V_Versorgung -> /ADC2_5V_Versorgung
- U106 pad 14: /Output_Schieber_DO -> /MOSI_Schieber_Daten_Out
- U106 pad 9: unconnected-(U106-QH'-Pad9) -> /7-Segment/Data
- U201 pad 10: Net-(RN202-R2.2) -> Net-(RN201-R4.2)
- U201 pad 2: Net-(RN202-R4.2) -> Net-(RN202-R1.2)
- U201 pad 3: Net-(RN201-R1.2) -> Net-(RN202-R2.2)
- U201 pad 4: Net-(RN201-R2.2) -> Net-(RN202-R3.2)
- U201 pad 6: Net-(RN201-R3.2) -> Net-(RN202-R4.2)
- U201 pad 7: Net-(RN201-R4.2) -> Net-(RN201-R1.2)
- U201 pad 8: Net-(RN202-R1.2) -> Net-(RN201-R2.2)
- U201 pad 9: Net-(RN202-R3.2) -> Net-(RN201-R3.2)
- U202 pad 14: /MOSI_Schieber_Daten_Out -> /7-Segment/Data
- U203 pad 10: Net-(RN204-R2.2) -> Net-(RN203-R4.2)
- U203 pad 2: Net-(RN204-R4.2) -> Net-(RN204-R1.2)
- U203 pad 3: Net-(RN203-R1.2) -> Net-(RN204-R2.2)
- U203 pad 4: Net-(RN203-R2.2) -> Net-(RN204-R3.2)
- U203 pad 6: Net-(RN203-R3.2) -> Net-(RN204-R4.2)
- U203 pad 7: Net-(RN203-R4.2) -> Net-(RN203-R1.2)
- U203 pad 8: Net-(RN204-R1.2) -> Net-(RN203-R2.2)
- U203 pad 9: Net-(RN204-R3.2) -> Net-(RN203-R3.2)
- U205 pad 10: Net-(RN206-R2.2) -> Net-(RN205-R4.2)
- U205 pad 2: Net-(RN206-R4.2) -> Net-(RN206-R1.2)
- U205 pad 3: Net-(RN205-R1.2) -> Net-(RN206-R2.2)
- U205 pad 4: Net-(RN205-R2.2) -> Net-(RN206-R3.2)
- U205 pad 6: Net-(RN205-R3.2) -> Net-(RN206-R4.2)
- U205 pad 7: Net-(RN205-R4.2) -> Net-(RN205-R1.2)
- U205 pad 8: Net-(RN206-R1.2) -> Net-(RN205-R2.2)
- U205 pad 9: Net-(RN206-R3.2) -> Net-(RN205-R3.2)
- U211 pad 4: Net-(RN212-R1.1) -> Net-(RN212-R4.1)
- U211 pad 5: Net-(RN212-R2.1) -> Net-(RN212-R3.1)
- U211 pad 6: Net-(RN212-R3.1) -> Net-(RN212-R2.1)
- U211 pad 7: Net-(RN212-R4.1) -> Net-(RN212-R1.1)
- U211 pad 9: /Output_Schieber_DO -> /7-Segment/DataOut
Routing:
- net +5V: track 0.00 -> 500.1 mm, vias 0 -> 23
- net +24V: track 0.00 -> 334.5 mm, vias 0 -> 4
- net /SS_Schieber_Latch: track 0.00 -> 265.3 mm, vias 0 -> 12
- net /OC1A_Dimmer: track 0.00 -> 260.9 mm, vias 0 -> 12
- net /SCK_Schieber_Takt: track 0.00 -> 259.8 mm, vias 0 -> 12
- net GNDA: track 0.00 -> 156.2 mm, vias 0 -> 5
- net GND: track 0.00 -> 129.1 mm, vias 0 -> 64
- net /ADC1_ID_2: track 0.00 -> 121.2 mm, vias 0 -> 2
- net /ADC0_ID_1: track 0.00 -> 112.8 mm, vias 0 -> 2
- net /ADC7_Messröhre 2 Signal: track 0.00 -> 97.6 mm, vias 0 -> 2
- net /ADC6_Messröhre 1 Signal: track 0.00 -> 96.5 mm, vias 0 -> 2
- net /7-Segment/Data: track 0.00 -> 90.0 mm, vias 0 -> 4
- net /R2_MagEn: track 0.00 -> 79.4 mm, vias 0 -> 2
- net /RS485_A: track 0.00 -> 71.9 mm, vias 0 -> 2
- net /R1_MagEn: track 0.00 -> 66.9 mm
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- added copper zone on F.Cu, net GND
Other:
- board outline added: 160 x 100 mm
