File: 03_Hardware/seg7.kicad_sch (KiCad schematic)
At the start: 50 parts, among them Q201 BC807, U201 8106BS, U202 74HC595, U203 8106BS, U204 74HC595, U205 8106BS, U206 74HC595, U207 5161BK, U208 74HC595, U209 74HC595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

Commit message: Software weitergemacht
Parts:
- C201, C202, C203, C204, C205, C206: footprint Resistor_SMD:R_0603_1608Metric -> Capacitor_SMD:C_0603_1608Metric
Changed lines of the file:
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@@
       (effects (font (size 1.27 1.27)) (justify left))
     )
-    (property "Footprint" "Resistor_SMD:R_0603_1608Metric" (at 102.5652 187.96 0)
+    (property "Footprint" "Capacitor_SMD:C_0603_1608Metric" (at 102.5652 187.96 0)
       (effects (font (size 1.27 1.27)) hide)
     )
@@
       (effects (font (size 1.27 1.27)) (justify left))
     )
-    (property "Footprint" "Resistor_SMD:R_0603_1608Metric" (at 51.7652 187.96 0)
+    (property "Footprint" "Capacitor_SMD:C_0603_1608Metric" (at 51.7652 187.96 0)
       (effects (font (size 1.27 1.27)) hide)
     )
@@
       (effects (font (size 1.27 1.27)) (justify left))
     )
-    (property "Footprint" "Resistor_SMD:R_0603_1608Metric" (at 89.8652 187.96 0)
+    (property "Footprint" "Capacitor_SMD:C_0603_1608Metric" (at 89.8652 187.96 0)
       (effects (font (size 1.27 1.27)) hide)
     )
@@
       (effects (font (size 1.27 1.27)) (justify left))
     )
-    (property "Footprint" "Resistor_SMD:R_0603_1608Metric" (at 39.0652 187.96 0)
+    (property "Footprint" "Capacitor_SMD:C_0603_1608Metric" (at 39.0652 187.96 0)
       (effects (font (size 1.27 1.27)) hide)
     )
@@
       (effects (font (size 1.27 1.27)) (justify left))
     )
-    (property "Footprint" "Resistor_SMD:R_0603_1608Metric" (at 64.4652 187.96 0)
+    (property "Footprint" "Capacitor_SMD:C_0603_1608Metric" (at 64.4652 187.96 0)
       (effects (font (size 1.27 1.27)) hide)
     )
@@
       (effects (font (size 1.27 1.27)) (justify left))
     )
-    (property "Footprint" "Resistor_SMD:R_0603_1608Metric" (at 77.1652 187.96 0)
-      (effects (font (size 1.27 1.27)) hide)
-    )
+    (property "Footprint" "Capacitor_SMD:C_0603_1608Metric" (at 77.1652 187.96 0)
+      (effects (font (size 1.27 1.27)) hide)
+    )
